Commit message: fix xacro files syntax and parameters so that the simulation can start properly. buoyancy has been added on all links but with wrong parameters. added thrusters with the visuals of airpropeller so simulate our motors.

File: usv_sim_lsa/usv_sim/urdf/athena_uwsim.urdf (robot description, URDF)
Before this commit: robot athena, 9 links, 8 joints
Links:
- link back_l_link: geometry visual mesh filename=meshes/naiad/backLeft.dae scale=0.21 0.21 0.21
- link back_r_link: geometry visual mesh filename=meshes/naiad/backRight.dae scale=0.21 0.21 0.21
- link base_link: geometry visual mesh filename=meshes/naiad/base_link.dae scale=0.21 0.21 0.21
- link center_r_link: geometry visual mesh filename=meshes/naiad/centerRight.dae scale=0.21 0.21 0.21
- link front_l_link: geometry visual mesh filename=meshes/naiad/frontLeft.dae scale=0.21 0.21 0.21
- link front_r_link: geometry visual mesh filename=meshes/naiad/frontRight.dae scale=0.21 0.21 0.21

File: usv_sim_lsa/usv_sim/xacro/athena.xacro (robot description, xacro)
@@ -28,5 +28,5 @@
     </gazebo>
     <!-- Define two steering thrusters, with assumed force control in Z-direction -->
-    <xacro:thruster_link name="fwd_left"  xyz="-0.3 0 -0.1" rpy="0 ${-PI/2-0.26} 0" rotationAxis="1 0 0" lowerLimit="0" upperLimit="0" parentLink="back_l_link"/>
-    <xacro:thruster_link name="fwd_right" xyz="-0.3 0 -0.1" rpy="0 ${-PI/2-0.26} 0" rotationAxis="1 0 0" lowerLimit="0" upperLimit="0" parentLink="back_r_link"/>
+    <xacro:thruster_link name="fwd_left"  xyz="0.005 0.0755 0" rpy="0 ${PI/2} 0" rotationAxis="1 0 0" lowerLimit="0" upperLimit="0" parentLink="base_link" thruster_scale="0.015"/>
+    <xacro:thruster_link name="fwd_right" xyz="0.005 -0.0755 0" rpy="0 ${PI/2} 0" rotationAxis="1 0 0" lowerLimit="0" upperLimit="0" parentLink="center_r_link" thruster_scale="0.015"/>
 </robot>

File: usv_sim_lsa/usv_sim/xacro/athena_subdivided_validated.xacro (robot description, xacro)
@@ -1,371 +1,373 @@
 <?xml version="1.0"?>
 <xacro xmlns:xacro="http://www.ros.org/wiki/xacro">
-    <xacro:property name="PI" value="3.1415926535897931"/>
-    <!-- Body properties -->
-    <xacro:property name="front_body_mass" value="0.5"/>
-    <xacro:property name="back_body_mass" value="2"/>
-    <xacro:property name="middle_body_mass" value="2"/>
-    <xacro:property name="back_water_displaced_mass" value="10"/>
-    <xacro:property name="middle_water_displaced_mass" value="10"/>
-    <xacro:property name="front_water_displaced_mass" value="5"/>
-    <xacro:property name="scale" value="0.21"/>
-    <xacro:property name="bl1" value=".1" />
-    <xacro:property name="bl2" value=".1" />
-    <link name="base_link">
-        <visual>
-          <origin rpy="0 0 0" xyz="0 0 0"/>
-          <geometry>
-            <mesh filename="package://usv_sim/meshes/naiad/base_link.dae" scale="${scale} ${scale} ${scale}"/>
-          </geometry>
-        </visual>
-        <collision>
-          <origin rpy="0 0 0" xyz="0 0 0"/>
-          <geometry>
-            <mesh filename="package://usv_sim/meshes/naiad/base_link.dae" scale="${scale} ${scale} ${scale}"/>
-          </geometry>
-        </collision>
-        <inertial>
-            <origin rpy="0 0 0" xyz="${0.35*scale} ${0.44*scale} ${-0.2*scale}"/>
-          <mass value="${middle_body_mass+extraPayload/2}"/>
-          <inertia ixx="0.1" ixy="0.0" ixz="0.0" iyy="1.4" iyz="0.0" izz="1.4"/>
-        </inertial>
-        <buoyancy>
-			<compensation>${middle_water_displaced_mass/middle_body_mass}</compensation>
-			<origin xyz="${0.35*scale} ${0.44*scale} ${-0.15*scale}"/>
-			<limit radius="0.1"/>
-			<damping rpy="${angularDampingXYZ}" xyz="${dampingXYZ}"/>
-         	<windVelocity>${windType}</windVelocity>
-			<frontal_area>0.0</frontal_area>
-			<lateral_area>0.012</lateral_area>
-			<lateral_length>1.06</lateral_length>
-	  		<waterVelocity>${waterType}</waterVelocity>
-        </buoyancy>
+  <xacro:property name="PI" value="3.1415926535897931"/>
+  <!-- Body properties -->
+  <xacro:property name="front_body_mass" value="0.5"/>
+  <xacro:property name="back_body_mass" value="2"/>
+  <xacro:property name="middle_body_mass" value="2"/>
+  <xacro:property name="back_water_displaced_mass" value="10"/>
+  <xacro:property name="middle_water_displaced_mass" value="10"/>
+  <xacro:property name="front_water_displaced_mass" value="5"/>
+  <xacro:property name="scale" value="0.21"/>
+  <xacro:property name="bl1" value=".1" />
+  <xacro:property name="bl2" value=".1" />
+  <link name='base_link'>
+    <pose frame=''>0 0 0 0 -0 0</pose>
+    <inertial>
+      <pose frame=''>0.0735 0.0924 -0.042 0 -0 0</pose>
+      <mass value="3.5"/>
+      <inertia ixx="0.1" ixy="0" ixz="0" iyy="1.4" iyz="0" izz="1.4"/>
+    </inertial>
+    <visual>
+      <pose frame=''>0 0 0 0 -0 0</pose>
+      <geometry>
+        <mesh filename="package://usv_sim/meshes/naiad/base_link.dae" scale="0.21 0.21 0.21" />
+      </geometry>
+    </visual>
+    <collision>
+      <pose frame=''>0 0 0 0 -0 0</pose>
+      <geometry>
+        <mesh filename="package://usv_sim/meshes/naiad/base_link.dae"/>
+      </geometry>
+    </collision>
+    <buoyancy>
+      <compensation>${middle_water_displaced_mass/middle_body_mass}</compensation>
+      <origin xyz="0 0 0"/>
+      <limit radius="0.1"/>
+      <damping rpy="${angularDampingXYZ}" xyz="${dampingXYZ}"/>
+      <windVelocity>${windType}</windVelocity>
+      <frontal_area>0.0</frontal_area>
+      <lateral_area>0.012</lateral_area>
+      <lateral_length>1.06</lateral_length>
+      <waterVelocity>${waterType}</waterVelocity>
+    </buoyancy>
+  </link>
+  <link name='back_l_link'>
+    <pose frame=''>0 0 0 0 -0 0</pose>
+    <inertial>
+      <pose frame=''>-0.126 0 -0.042 0 -0 0</pose>
+      <mass value="2"/>
+      <inertia ixx="0.1" ixy="0" ixz="0" iyy="1.4" iyz="0" izz="1.4"/>
+    </inertial>
+    <visual>
+      <pose frame=''>0 0 0 0 -0 0</pose>
+      <geometry>
+        <mesh filename="package://usv_sim/meshes/naiad/backLeft.dae" scale="0.21 0.21 0.21"/>
+      </geometry>
+    </visual>
+    <collision>
+      <pose frame=''>0 0 0 0 -0 0</pose>
+      <geometry>
+        <mesh filename="package://usv_sim/meshes/naiad/backLeft.dae" />
+      </geometry>
+    </collision>
+    <buoyancy>
+      <compensation>${back_water_displaced_mass/back_body_mass}</compensation>
+      <origin xyz="0 0 0"/>
+      <limit radius="0.1"/>
+      <damping rpy="${angularDampingXYZ}" xyz="${dampingXYZ}"/>
+      <windVelocity>${windType}</windVelocity>
+      <frontal_area>0.0</frontal_area>
+      <lateral_area>0.012</lateral_area>
+      <lateral_length>1.06</lateral_length>
+      <waterVelocity>${waterType}</waterVelocity>
+    </buoyancy>
+  </link>
+  <link name='back_r_link'>
+    <pose frame=''>0 0 0 0 -0 0</pose>
+    <inertial>
+      <pose frame=''>-0.126 0 -0.042 0 -0 0</pose>
+      <mass value="2"/>
+      <inertia ixx="0.1" ixy="0" ixz="0" iyy="1.4" iyz="0" izz="1.4"/>
+    </inertial>
+    <visual>
+      <pose frame=''>0 0 0 0 -0 0</pose>
+      <geometry>
+        <mesh filename="package://usv_sim/meshes/naiad/backRight.dae" scale="0.21 0.21 0.21"/>
+      </geometry>
+    </visual>
+    <collision>
+      <pose frame=''>0 0 0 0 -0 0</pose>
+      <geometry>
+        <mesh filename="package://usv_sim/meshes/naiad/backRight.dae" />
+      </geometry>
+    </collision>
+    <buoyancy>
+      <compensation>${back_water_displaced_mass/back_body_mass}</compensation>
+      <origin xyz="0 0 0"/>
+      <limit radius="0.1"/>
+      <damping rpy="${angularDampingXYZ}" xyz="${dampingXYZ}"/>
+      <windVelocity>${windType}</windVelocity>
+      <frontal_area>0.0</frontal_area>
+      <lateral_area>0.012</lateral_area>
+      <lateral_length>1.06</lateral_length>
+      <waterVelocity>${waterType}</waterVelocity>
+    </buoyancy>
+  </link>
+  <link name='center_r_link'>
+    <pose frame=''>0 0 0 0 -0 0</pose>
+    <inertial>
+      <pose frame=''>0.0735 -0.0924 -0.042 0 -0 0</pose>
+      <mass value="3.5"/>
+      <inertia ixx="0.1" ixy="0" ixz="0" iyy="1.4" iyz="0" izz="1.4"/>
+    </inertial>
+    <visual>
+      <pose frame=''>0 0 0 0 -0 0</pose>
+      <geometry>
+        <mesh filename="package://usv_sim/meshes/naiad/centerRight.dae" scale="0.21 0.21 0.21"/>
+      </geometry>
+    </visual>
+    <collision>
+      <pose frame=''>0 0 0 0 -0 0</pose>
+      <geometry>
+        <mesh filename="package://usv_sim/meshes/naiad/centerRight.dae" />
+      </geometry>
+    </collision>
+    <buoyancy>
+      <compensation>${middle_water_displaced_mass/middle_body_mass}</compensation>
+      <origin xyz="0 0 0"/>
+      <limit radius="0.1"/>
+      <damping rpy="${angularDampingXYZ}" xyz="${dampingXYZ}"/>
+      <windVelocity>${windType}</windVelocity>
+      <frontal_area>0.0</frontal_area>
+      <lateral_area>0.012</lateral_area>
+      <lateral_length>1.06</lateral_length>
+      <waterVelocity>${waterType}</waterVelocity>
+    </buoyancy>
+  </link>
+  <link name='front_l_link'>
+    <pose frame=''>0 0 0 0 -0 0</pose>
+    <inertial>
+      <pose frame=''>0.084 0 -0.021 0 -0 0</pose>
+      <mass value="0.5"/>
+      <inertia ixx="0.1" ixy="0" ixz="0" iyy="1.4" iyz="0" izz="1.4"/>
+    </inertial>
+    <visual>
+      <pose frame=''>0 0 0 0 -0 0</pose>
+      <geometry>
+        <mesh filename="package://usv_sim/meshes/naiad/frontLeft.dae" scale="0.21 0.21 0.21"/>
+      </geometry>
+    </visual>
+    <collision>
+      <pose frame=''>0 0 0 0 -0 0</pose>
+      <geometry>
+        <mesh filename="package://usv_sim/meshes/naiad/frontLeft.dae" />
+      </geometry>
+    </collision>
+    <buoyancy>
+      <compensation>${front_water_displaced_mass/front_body_mass}</compensation>
+      <origin xyz="0 0 0"/>
+      <limit radius="0.1"/>
+      <damping rpy="${angularDampingXYZ}" xyz="${dampingXYZ}"/>
+      <windVelocity>${windType}</windVelocity>
+      <frontal_area>0.0</frontal_area>
+      <lateral_area>0.012</lateral_area>
+      <lateral_length>1.06</lateral_length>
+      <waterVelocity>${waterType}</waterVelocity>
+    </buoyancy>
+  </link>
+  <link name='front_r_link'>
+    <pose frame=''>0 0 0 0 -0 0</pose>
+    <inertial>
+      <pose frame=''>0.084 0 -0.021 0 -0 0</pose>
+      <mass value="0.5"/>
+      <inertia ixx="0.1" ixy="0" ixz="0" iyy="1.4" iyz="0" izz="1.4"/>
+    </inertial>
+    <visual>
+      <pose frame=''>0 0 0 0 -0 0</pose>
+      <geometry>
+        <mesh filename="package://usv_sim/meshes/naiad/frontRight.dae" scale="0.21 0.21 0.21"/>
+      </geometry>
+    </visual>
+    <collision>
+      <pose frame=''>0 0 0 0 -0 0</pose>
+      <geometry>
+        <mesh filename="package://usv_sim/meshes/naiad/frontRight.dae" />
+      </geometry>
+    </collision>
+    <buoyancy>
+      <compensation>${front_water_displaced_mass/front_body_mass}</compensation>
+      <origin xyz="0 0 0"/>
+      <limit radius="0.1"/>
+      <damping rpy="${angularDampingXYZ}" xyz="${dampingXYZ}"/>
+      <windVelocity>${windType}</windVelocity>
+      <frontal_area>0.0</frontal_area>
+      <lateral_area>0.012</lateral_area>
+      <lateral_length>1.06</lateral_length>
+      <waterVelocity>${waterType}</waterVelocity>
+    </buoyancy>
+  </link>
+  <!--
+    <link name='fwd_left'>
+    <pose frame=''>0.053619 0.043999 -0.1 3.14159 -1.3108 3.14159</pose>
+    <inertial>
+    <pose frame=''>-0.042 0 0.063 0 -0 0</pose>
+    <mass value="0.1"/>
+    <inertia ixx="0.1" ixy="0" ixz="0" iyy="0.1" iyz="0" izz="0.1"/>
+    </inertial>
+    <visual>
+    <pose frame=''>-0.0315 0 0 0 -0 0</pose>
+    <geometry>
+    <mesh filename="package://usv_sim/meshes/simpleHull3/thruster.dae" scale="0.21 0.21 0.21"/>
+    </geometry>
+    </visual>
+    <collision>
+    <pose frame=''>-0.0315 0 0 0 -0 0</pose>
+    <geometry>
+    <mesh filename="package://usv_sim/meshes/simpleHull3/thruster.dae" />
+    </geometry>
+    </collision>
     </link>
-    <link name="center_r_link">
-    	<visual>
-          <origin rpy="0 0 0"  xyz="0 0 ${0*scale}"/>
-          <geometry>
-            <mesh filename="package://usv_sim/meshes/naiad/centerRight.dae" scale="${scale} ${scale} ${scale}"/>
-          </geometry>
-        </visual>
-        <collision>
-          <origin rpy="0 0 0"  xyz="0 0 ${0*scale}"/>
-          <geometry>
-           	<mesh filename="package://usv_sim/meshes/naiad/centerRight.dae" scale="${scale} ${scale} ${scale}"/>
-          </geometry>
-        </collision>
-        <inertial>
-            <origin rpy="0 0 0" xyz="${0.35*scale} ${-0.44*scale} ${-0.2*scale}"/>
-          <mass value="${middle_body_mass+extraPayload/2}"/>
-          <inertia ixx="0.1" ixy="0.0" ixz="0.0" iyy="1.4" iyz="0.0" izz="1.4"/>
-        </inertial>
-        <buoyancy>
-          <compensation>${middle_water_displaced_mass/middle_body_mass}</compensation>
-          <origin xyz="${0.35*scale} ${-0.44*scale} ${-0.15*scale}"/>
-          <limit radius="0.1"/>
-          <damping rpy="${angularDampingXYZ}" xyz="${dampingXYZ}"/>
-			<windVelocity>${windType}</windVelocity>
-			<frontal_area>0.0</frontal_area>
-			<lateral_area>0.012</lateral_area>
-			<lateral_length>1.06</lateral_length>
-	  <waterVelocity>${waterType}</waterVelocity>
-        </buoyancy>
+    <link name='fwd_right'>
+    <pose frame=''>0.053604 -0.04615 -0.1 3.14159 -1.3108 3.14159</pose>
+    <inertial>
+    <pose frame=''>-0.042 0 0.063 0 -0 0</pose>
+    <mass value="0.1"/>
+    <inertia ixx="0.1" ixy="0" ixz="0" iyy="0.1" iyz="0" izz="0.1"/>
+    </inertial>
+    <visual>
+    <pose frame=''>-0.0315 0 0 0 -0 0</pose>
+    <geometry>
+    <mesh filename="package://usv_sim/meshes/simpleHull3/thruster.dae" scale="0.21 0.21 0.21"/>
+    </geometry>
+    </visual>
+    <collision>
+    <pose frame=''>-0.0315 0 0 0 -0 0</pose>
+    <geometry>
+    <mesh filename="package://usv_sim/meshes/simpleHull3/thruster.dae"/>
+    </geometry>
+    </collision>
     </link>
-    <joint name="center_r_joint" type="revolute">
-        <parent link="base_link"/>
-        <child link="center_r_link"/>
-        <origin rpy="0 0 0" xyz="0 0 0"/>
-	<limit effort="50" velocity="5" lower="0" upper="0" />
-            <dynamics damping="1.0"/>
-            <axis xyz="1 0 0"/>
-    </joint>
-    <link name="back_l_link">
-        <visual>
-          <origin rpy="0 0 0"  xyz="0 0 0"/>
-          <geometry>
-           	<mesh filename="package://usv_sim/meshes/naiad/backLeft.dae" scale="${scale} ${scale} ${scale}"/>
-          </geometry>
-        </visual>
-        <collision>
-          <origin rpy="0 0 0"  xyz="0 0 0"/>
-          <geometry>
-           	<mesh filename="package://usv_sim/meshes/naiad/backLeft.dae" scale="${scale} ${scale} ${scale}"/>
-          </geometry>
-        </collision>
-        <inertial>
-            <origin rpy="0 0 0" xyz="${-0.6*scale} 0 ${-0.2*scale}"/>
-          <mass value="${back_body_mass}"/>
-          <inertia ixx="0.1" ixy="0.0" ixz="0.0" iyy="1.4" iyz="0.0" izz="1.4"/>
-        </inertial>
-        <buoyancy>
-			<compensation>${back_water_displaced_mass/back_body_mass}</compensation>
-			<origin xyz="${-0.6*scale} 0 ${-0.15*scale}"/>
-			<limit radius="0.1"/>
-			<damping rpy="${angularDampingXYZ}" xyz="${dampingXYZ}"/>
-			<windVelocity>${windType}</windVelocity>
-			<frontal_area>0.02</frontal_area>
-			<lateral_area>0.012</lateral_area>
-			<lateral_length>1.06</lateral_length>
-	  		<waterVelocity>${waterType}</waterVelocity>
-        </buoyancy>
-    </link>
-    <joint name="back_l_joint" type="revolute">
-        <parent link="base_link"/>
-        <child link="back_l_link"/>
-        <origin rpy="0 0 0" xyz="${-0.5*scale} ${0.39*scale} 0"/>
-	<limit effort="50" velocity="5" lower="0" upper="0" />
-            <dynamics damping="1.0"/>
-            <axis xyz="1 0 0"/>
-    </joint>
-    <link name="back_r_link">
-    	<visual>
-          <origin rpy="0 0 0"  xyz="0 0 0"/>
-          <geometry>
-           	<mesh filename="package://usv_sim/meshes/naiad/backRight.dae" scale="${scale} ${scale} ${scale}"/>
-          </geometry>
-    	</visual>
-        <collision>
-          <origin rpy="0 0 0"  xyz="0 0 0"/>
-          <geometry>
-           	<mesh filename="package://usv_sim/meshes/naiad/backRight.dae" scale="${scale} ${scale} ${scale}"/>
-          </geometry>
-        </collision>
-        <inertial>
-            <origin rpy="0 0 0" xyz="${-0.6*scale} 0 ${-0.2*scale}"/>
-          <mass value="${back_body_mass}"/>
-          <inertia ixx="0.1" ixy="0.0" ixz="0.0" iyy="1.4" iyz="0.0" izz="1.4"/>
-        </inertial>
-        <buoyancy>
-          	<compensation>${back_water_displaced_mass/back_body_mass}</compensation>
-          	<origin xyz="${-0.6*scale} 0 ${-0.15*scale}"/>
-          	<limit radius="0.1"/>
-          	<damping rpy="${angularDampingXYZ}" xyz="${dampingXYZ}"/>
-          	<windVelocity>${windType}</windVelocity>
-			<frontal_area>0.02</frontal_area>
-			<lateral_area>0.012</lateral_area>
-			<lateral_length>1.06</lateral_length>
-	  		<waterVelocity>${waterType}</waterVelocity>
-        </buoyancy>
-    </link>
-    <joint name="back_r_joint" type="revolute">
-        <parent link="base_link"/>
-        <child link="back_r_link"/>
-        <origin rpy="0 0 0" xyz="${-0.5*scale} ${-0.39*scale} 0"/>
-	<limit effort="50" velocity="5" lower="0" upper="0" />
-            <dynamics damping="1.0"/>
-            <axis xyz="1 0 0"/>
-    </joint>
-    <link name="front_l_link">
-    	<visual>
-    	<origin rpy="0 0 0"  xyz="0 0 0"/>
-          <geometry>
-           	<mesh filename="package://usv_sim/meshes/naiad/frontLeft.dae" scale="${scale} ${scale} ${scale}"/>
-          </geometry>
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