Commit message: fixes on athena floating dynamics and motor positioning

File: athena_description/urdf/core.urdf.xacro (robot description, xacro)
@@ -14,5 +14,5 @@
   </link>
   <!-- Robot mesh -->
-  <xacro:add_to_base_link element="base" mesh="package://athena_description/meshes/athena.dae">
+  <xacro:add_to_base_link element="base" mesh="package://athena_description/meshes/athena.obj">
     <origin rpy="-1.57 0 3.14" xyz="0.7 0 0.4"/>
   </xacro:add_to_base_link>
@@ -35,25 +35,9 @@
   <!-- thruster_0 -->
   <xacro:add_to_base_link_no_mesh element="thruster_0">
-    <origin rpy="0.0 0.0 -1.571" xyz="-0.38 0.0576 0.0"/>
+    <origin rpy="0.0 0.0 -1.571" xyz="0.22 -0.11 0.15"/>
   </xacro:add_to_base_link_no_mesh>
   <!-- thruster_1 -->
   <xacro:add_to_base_link_no_mesh element="thruster_1">
-    <origin rpy="0.0 0.0 -1.571" xyz="0.38 0.0576 0.0"/>
-  </xacro:add_to_base_link_no_mesh>
-  <!-- thruster_2 -->
-  <xacro:add_to_base_link_no_mesh element="thruster_2">
-    <origin rpy="0.0 1.571 0.0" xyz="-0.24 0.445 0.0"/>
-  </xacro:add_to_base_link_no_mesh>
-  <!-- thruster_3 -->
-  <xacro:add_to_base_link_no_mesh element="thruster_3">
-    <origin rpy="0.0 1.571 0.0" xyz="0.24 0.445 0.0"/>
-  </xacro:add_to_base_link_no_mesh>
-  <!-- thruster_4 -->
-  <xacro:add_to_base_link_no_mesh element="thruster_4">
-    <origin rpy="0.0 1.571 3.1416" xyz="-0.24 -0.445 0.0"/>
-  </xacro:add_to_base_link_no_mesh>
-  <!-- thruster_5 -->
-  <xacro:add_to_base_link_no_mesh element="thruster_5">
-    <origin rpy="0.0 1.571 3.1416" xyz="0.24 -0.445 0.0"/>
+    <origin rpy="0.0 0.0 -1.571" xyz="-0.22 -0.11 0.15"/>
   </xacro:add_to_base_link_no_mesh>
 </robot>
